File: pcb/MainBoard/MainBoard.kicad_pcb (KiCad board)
At the start: 2 copper layers, 1 part

Commit message: updated to the main board
Parts:
- added REF**: JST_EH_B3B-EH-A_1x03_P2.50mm_Vertical, Connector_JST:JST_EH_B3B-EH-A_1x03_P2.50mm_Vertical, F.Cu at (176.5, 48.3)
- added REF**: JST_EH_B3B-EH-A_1x03_P2.50mm_Vertical, Connector_JST:JST_EH_B3B-EH-A_1x03_P2.50mm_Vertical, F.Cu at (142.2, 68.6)
- added REF**: JST_EH_B3B-EH-A_1x03_P2.50mm_Vertical, Connector_JST:JST_EH_B3B-EH-A_1x03_P2.50mm_Vertical, F.Cu at (153.7, 57.1)
- added REF**: JST_EH_B3B-EH-A_1x03_P2.50mm_Vertical, Connector_JST:JST_EH_B3B-EH-A_1x03_P2.50mm_Vertical, F.Cu at (142.2, 62.2)
- added REF**: JST_EH_B3B-EH-A_1x03_P2.50mm_Vertical, Connector_JST:JST_EH_B3B-EH-A_1x03_P2.50mm_Vertical, F.Cu at (142.2, 57.1)
- added REF**: JST_EH_B3B-EH-A_1x03_P2.50mm_Vertical, Connector_JST:JST_EH_B3B-EH-A_1x03_P2.50mm_Vertical, F.Cu at (176.5, 57.1)
- added REF**: JST_EH_B3B-EH-A_1x03_P2.50mm_Vertical, Connector_JST:JST_EH_B3B-EH-A_1x03_P2.50mm_Vertical, F.Cu at (176.5, 66.0)
- added REF**: JST_EH_B3B-EH-A_1x03_P2.50mm_Vertical, Connector_JST:JST_EH_B3B-EH-A_1x03_P2.50mm_Vertical, F.Cu at (176.5, 81.3)
- added REF**: JST_EH_B3B-EH-A_1x03_P2.50mm_Vertical, Connector_JST:JST_EH_B3B-EH-A_1x03_P2.50mm_Vertical, F.Cu at (176.5, 73.7)
- added REF**: JST_EH_B3B-EH-A_1x03_P2.50mm_Vertical, Connector_JST:JST_EH_B3B-EH-A_1x03_P2.50mm_Vertical, F.Cu at (167.6, 39.4)
- added REF**: JST_EH_B3B-EH-A_1x03_P2.50mm_Vertical, Connector_JST:JST_EH_B3B-EH-A_1x03_P2.50mm_Vertical, F.Cu at (156.2, 63.5)
- added REF**: JST_EH_B3B-EH-A_1x03_P2.50mm_Vertical, Connector_JST:JST_EH_B3B-EH-A_1x03_P2.50mm_Vertical, F.Cu at (154.9, 49.5)
- added REF**: JST_EH_B3B-EH-A_1x03_P2.50mm_Vertical, Connector_JST:JST_EH_B3B-EH-A_1x03_P2.50mm_Vertical, F.Cu at (142.2, 49.5)
