File: pcb/RedLegs_pwrbrd/RedLegs_pwrbrd.kicad_pcb (KiCad board)
At the start: 2 copper layers, 30 parts, among them J1 Conn_01x02, J10 Conn_01x02, J11 Conn_01x02, J12 Conn_01x02, J2 Conn_01x02, J3 Conn_01x02, J4 Conn_01x02, J5 Conn_01x02, J6 Conn_01x02, J7 Conn_01x02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

Commit message: Finish power board
Parts:
- added Mnt_Hole: M4, MountingHole:MountingHole_4.3mm_M4, F.Cu at (191.8, 59.7)
- added REF**: M4, MountingHole:MountingHole_4.3mm_M4, F.Cu at (119.4, 142.2)
- added REF**: M4, MountingHole:MountingHole_4.3mm_M4, F.Cu at (189.2, 142.2)
- added REF**: M4, MountingHole:MountingHole_4.3mm_M4, F.Cu at (118.1, 59.7)
- H1: value Battery_Positive -> BATT_VCC
- H2: value Battery_Ground -> BATT_GND
- moved H2 8.04 mm to (130.8, 59.7)
- moved R1 5.24 mm to (183.1, 63.5)
- moved D1 5.08 mm to (181.6, 58.4)
- moved H1 5.08 mm to (143.5, 59.7)
- moved U1 2.97 mm to (173.6, 59.7)
- moved F0 2.54 mm to (152.4, 58.1)
Routing:
- net GND: track 312.1 -> 13.8 mm
- net VCC: track 274.5 -> 270.6 mm
- net Net-(R1-Pad2): track 16.5 -> 13.7 mm
- net +BATT: track 10.1 -> 7.74 mm
- net Net-(D1-Pad2): track 6.35 -> 5.08 mm
- added copper zone on B.Cu, net GND
Other:
- board outline added: 87.6 x 96.5 mm
- board text added: "+"
- board text added: "-"
- board text added: "Red Legs Power Board - Mk I 2020"
